Commit message: feat: update anchor geometry to 3-ceiling/2-floor layout, add furniture to Sionna scene
Anchors: a0-a2 ceiling corners/mid at z=2.7, a3-a4 floor mid-walls at z=0.3.
Sionna scene: add ITU-wood furniture AABB boxes (bookshelf, cafe_table, cabinet)
matching room.world.xacro model poses. PLY normals verified outward by cross-product.

Co-Authored-By: Claude Sonnet 4.6 <noreply@anthropic.com>

File: src/microuwb_gazebo/worlds/room.world.xacro (robot description, xacro)
@@ -130,80 +130,80 @@
     </xacro:if>
     <!-- ───────────────── UWB ANCHORS ───────────────── -->
-    <!-- a0: SW corner high -->
+    <!-- a0: SW ceiling corner -->
     <model name="anchor_0">
       <static>true</static>
-      <pose>0.1 0.1 2.5 0 0 0</pose>
-      <link name="link">
-        <visual name="body">
-          <geometry><cylinder><radius>0.03</radius><length>0.05</length></cylinder></geometry>
-          <material>
-            <ambient>1.0 0.0 0.0 1.0</ambient>
-            <diffuse>1.0 0.0 0.0 1.0</diffuse>
-            <emissive>0.8 0.0 0.0 1.0</emissive>
-          </material>
-        </visual>
-        <collision name="collision">
-          <geometry><cylinder><radius>0.03</radius><length>0.05</length></cylinder></geometry>
-        </collision>
-      </link>
-    </model>
-    <!-- a1: SE corner high -->
+      <pose>0.1 0.1 2.7 0 0 0</pose>
+      <link name="link">
+        <visual name="body">
+          <geometry><cylinder><radius>0.03</radius><length>0.05</length></cylinder></geometry>
+          <material>
+            <ambient>1.0 0.0 0.0 1.0</ambient>
+            <diffuse>1.0 0.0 0.0 1.0</diffuse>
+            <emissive>0.8 0.0 0.0 1.0</emissive>
+          </material>
+        </visual>
+        <collision name="collision">
+          <geometry><cylinder><radius>0.03</radius><length>0.05</length></cylinder></geometry>
+        </collision>
+      </link>
+    </model>
+    <!-- a1: SE ceiling corner -->
     <model name="anchor_1">
       <static>true</static>
-      <pose>4.9 0.1 2.5 0 0 0</pose>
-      <link name="link">
-        <visual name="body">
-          <geometry><cylinder><radius>0.03</radius><length>0.05</length></cylinder></geometry>
-          <material>
-            <ambient>1.0 0.0 0.0 1.0</ambient>
-            <diffuse>1.0 0.0 0.0 1.0</diffuse>
-            <emissive>0.8 0.0 0.0 1.0</emissive>
-          </material>
-        </visual>
-        <collision name="collision">
-          <geometry><cylinder><radius>0.03</radius><length>0.05</length></cylinder></geometry>
-        </collision>
-      </link>
-    </model>
-    <!-- a2: NW corner high -->
+      <pose>4.9 0.1 2.7 0 0 0</pose>
+      <link name="link">
+        <visual name="body">
+          <geometry><cylinder><radius>0.03</radius><length>0.05</length></cylinder></geometry>
+          <material>
+            <ambient>1.0 0.0 0.0 1.0</ambient>
+            <diffuse>1.0 0.0 0.0 1.0</diffuse>
+            <emissive>0.8 0.0 0.0 1.0</emissive>
+          </material>
+        </visual>
+        <collision name="collision">
+          <geometry><cylinder><radius>0.03</radius><length>0.05</length></cylinder></geometry>
+        </collision>
+      </link>
+    </model>
+    <!-- a2: ceiling mid north wall -->
     <model name="anchor_2">
       <static>true</static>
-      <pose>0.1 3.9 2.5 0 0 0</pose>
-      <link name="link">
-        <visual name="body">
-          <geometry><cylinder><radius>0.03</radius><length>0.05</length></cylinder></geometry>
-          <material>
-            <ambient>1.0 0.0 0.0 1.0</ambient>
-            <diffuse>1.0 0.0 0.0 1.0</diffuse>
-            <emissive>0.8 0.0 0.0 1.0</emissive>
-          </material>
-        </visual>
-        <collision name="collision">
-          <geometry><cylinder><radius>0.03</radius><length>0.05</length></cylinder></geometry>
-        </collision>
-      </link>
-    </model>
-    <!-- a3: NE corner high -->
+      <pose>2.5 3.9 2.7 0 0 0</pose>
+      <link name="link">
+        <visual name="body">
+          <geometry><cylinder><radius>0.03</radius><length>0.05</length></cylinder></geometry>
+          <material>
+            <ambient>1.0 0.0 0.0 1.0</ambient>
+            <diffuse>1.0 0.0 0.0 1.0</diffuse>
+            <emissive>0.8 0.0 0.0 1.0</emissive>
+          </material>
+        </visual>
+        <collision name="collision">
+          <geometry><cylinder><radius>0.03</radius><length>0.05</length></cylinder></geometry>
+        </collision>
+      </link>
+    </model>
+    <!-- a3: floor mid west wall -->
     <model name="anchor_3">
       <static>true</static>
-      <pose>4.9 3.9 2.5 0 0 0</pose>
-      <link name="link">
-        <visual name="body">
-          <geometry><cylinder><radius>0.03</radius><length>0.05</length></cylinder></geometry>
-          <material>
-            <ambient>1.0 0.0 0.0 1.0</ambient>
-            <diffuse>1.0 0.0 0.0 1.0</diffuse>
-            <emissive>0.8 0.0 0.0 1.0</emissive>
-          </material>
-        </visual>
-        <collision name="collision">
-          <geometry><cylinder><radius>0.03</radius><length>0.05</length></cylinder></geometry>
-        </collision>
-      </link>
-    </model>
-    <!-- a4: centre overhead -->
+      <pose>0.1 2.0 0.3 0 0 0</pose>
+      <link name="link">
+        <visual name="body">
+          <geometry><cylinder><radius>0.03</radius><length>0.05</length></cylinder></geometry>
+          <material>
+            <ambient>1.0 0.0 0.0 1.0</ambient>
+            <diffuse>1.0 0.0 0.0 1.0</diffuse>
+            <emissive>0.8 0.0 0.0 1.0</emissive>
+          </material>
+        </visual>
+        <collision name="collision">
+          <geometry><cylinder><radius>0.03</radius><length>0.05</length></cylinder></geometry>
+        </collision>
+      </link>
+    </model>
+    <!-- a4: floor mid east wall -->
     <model name="anchor_4">
       <static>true</static>
-      <pose>2.5 2.0 2.8 0 0 0</pose>
+      <pose>4.9 2.0 0.3 0 0 0</pose>
       <link name="link">
         <visual name="body">
